File: hardware/red-blink.kicad_pcb (KiCad board)
At the start: 2 copper layers, 33 x 33 mm, 7 parts, among them J1 Conn_01x03_Male, U1 ATtiny402-SS

Commit message: Working on PCB Layout
Parts:
- added D1: LED, janis:LED_2214A, F.Cu at (150.5, 90.3)
- added D2: LED, janis:LED_2214A, F.Cu at (157.0, 79.0)
- added D3: LED, janis:LED_2214A, F.Cu at (137.5, 90.3)
- added D4: LED, janis:LED_2214A, F.Cu at (137.5, 67.7)
- added D5: LED, janis:LED_2214A, F.Cu at (150.5, 67.7)
- added D6: LED, janis:LED_2214A, F.Cu at (131.0, 79.0)
- moved J1 27.1 mm to (161.0, 91.5)
- moved R1 2.24 mm to (139.0, 80.0), turned to 90 degrees
- moved R3 2.24 mm to (149.0, 77.0), turned to 270 degrees
- moved R2 2.00 mm to (149.0, 81.0), turned to 90 degrees

Commit message: Finished schematic and PCB
Parts:
- removed J1: Conn_01x03_Male, Connector_PinSocket_2.54mm:PinSocket_1x03_P2.54mm_Vertical
- added C2: 10uF, Capacitor_SMD:C_0805_2012Metric, F.Cu at (135.0, 79.0)
- added C3: 10uF, Capacitor_SMD:C_0805_2012Metric, F.Cu at (153.0, 79.0)
- added CON1: 1PIN, Raksts_Test:TestPoint_2.00mm, F.Cu at (147.0, 85.5)
- added CON2: 1PIN, Raksts_Test:TestPoint_2.00mm, F.Cu at (144.0, 85.5)
- added CON3: 1PIN, Raksts_Test:TestPoint_2.00mm, F.Cu at (141.0, 85.5)
- added CON4: 1PIN, Raksts_Test:TestPoint_2.00mm, F.Cu at (138.0, 85.5)
- added SW1: SWT-2, Button_Switch_SMD:SW_SPST_EVQQ2, F.Cu at (144.0, 79.0)
- D1, D2, D3, D4, D5, D6: footprint janis:LED_2214A -> janis:LED_3528
- moved D4 13.0 mm to (150.5, 67.7), turned to 240 degrees
- moved D5 13.0 mm to (137.5, 67.7), turned to 120 degrees
- moved U1 7.00 mm to (144.0, 72.0)
- moved C1 6.71 mm to (138.0, 72.0), turned to 180 degrees
- moved R2 6.58 mm to (150.0, 74.5), turned to 180 degrees
- moved R1 5.59 mm to (138.0, 74.5), turned to 0 degrees
- moved R3 5.10 mm to (150.0, 72.0), turned to 180 degrees
Routing:
- net Net-(D1-Pad2): track 0.00 -> 61.9 mm
- net Net-(D2-Pad1): track 0.00 -> 49.0 mm
- net Net-(D1-Pad1): track 0.00 -> 41.5 mm
- net Net-(BT1-Pad1): track 0.00 -> 28.5 mm, vias 0 -> 2
- net Net-(CON2-Pad1): track 0.00 -> 22.9 mm
- net Net-(CON4-Pad1): track 0.00 -> 18.2 mm
- net Net-(SW1-Pad1): track 0.00 -> 14.2 mm
- net Net-(R3-Pad2): track 0.00 -> 2.85 mm
- net Net-(R2-Pad2): track 0.00 -> 2.83 mm
- net Net-(R1-Pad2): track 0.00 -> 2.83 mm
- net GND: vias 0 -> 20
- added copper zone on B.Cu, net GND
- added copper zone on F.Cu, net GND
Other:
- board text added: "2019"
- board text added: "3V"
- board text added: "GND"
- board text added: "GPIO"
- board text added: "RV1G Robotics Club"
- board text added: "Red Blink"
- board text added: "TPI"
