File: hardware/red-blink.sch (KiCad schematic (older format))
At the start: 13 parts

Commit message: Working on PCB Layout
Parts:
- BT1: renamed from BT?; footprint (none) -> Battery:BatteryHolder_Keystone_3002_1x2032
- C1: renamed from C?; footprint (none) -> Capacitor_SMD:C_0805_2012Metric
- D1, D2, D3, D4, D5, D6: renamed from D?; footprint (none) -> janis:LED_2214A
- J1: renamed from J?; footprint (none) -> Connector_PinSocket_2.54mm:PinSocket_1x03_P2.54mm_Vertical
- R1, R2, R3: renamed from R?; footprint (none) -> Resistor_SMD:R_0805_2012Metric
- gave numbers to parts that had none: 1
Changed lines of the file:
@@
 $EndDescr
 $Comp
-L MCU_Microchip_ATtiny:ATtiny402-SS U?
+L MCU_Microchip_ATtiny:ATtiny402-SS U1
 U 1 1 5DC981FC
 P 5700 3500
-F 0 "U?" H 5171 3546 50  0000 R CNN
+F 0 "U1" H 5171 3546 50  0000 R CNN
 F 1 "ATtiny402-SS" H 5171 3455 50  0000 R CNN
 F 2 "Package_SO:SOIC-8_3.9x4.9mm_P1.27mm" H 5700 3500 50  0001 C CIN
@@
 $EndComp
 $Comp
-L Device:Battery_Cell BT?
+L Device:Battery_Cell BT1
 U 1 1 5DC992B0
 P 3800 3500
-F 0 "BT?" H 3918 3596 50  0000 L CNN
+F 0 "BT1" H 3918 3596 50  0000 L CNN
 F 1 "Battery_Cell" H 3918 3505 50  0000 L CNN
-F 2 "" V 3800 3560 50  0001 C CNN
+F 2 "Battery:BatteryHolder_Keystone_3002_1x2032" V 3800 3560 50  0001 C CNN
 F 3 "~" V 3800 3560 50  0001 C CNN
 	1    3800 3500
@@
 $EndComp
 $Comp
-L Device:C_Small C?
+L Device:C_Small C1
 U 1 1 5DC999E0
 P 4500 3000
-F 0 "C?" H 4592 3046 50  0000 L CNN
+F 0 "C1" H 4592 3046 50  0000 L CNN
 F 1 "0.1uF" H 4592 2955 50  0000 L CNN
-F 2 "" H 4500 3000 50  0001 C CNN
+F 2 "Capacitor_SMD:C_0805_2012Metric" H 4500 3000 50  0001 C CNN
 F 3 "~" H 4500 3000 50  0001 C CNN
 	1    4500 3000
@@
 	4500 3100 4500 3200
 $Comp
-L power:GND #PWR?
+L power:GND #PWR0101
 U 1 1 5DC9A9DB
 P 4500 3200
-F 0 "#PWR?" H 4500 2950 50  0001 C CNN
+F 0 "#PWR0101" H 4500 2950 50  0001 C CNN
 F 1 "GND" H 4505 3027 50  0000 C CNN
 F 2 "" H 4500 3200 50  0001 C CNN
@@
 $EndComp
 $Comp
-L power:GND #PWR?
+L power:GND #PWR0102
 U 1 1 5DC9AD2E
 P 5700 4300
-F 0 "#PWR?" H 5700 4050 50  0001 C CNN
+F 0 "#PWR0102" H 5700 4050 50  0001 C CNN
 F 1 "GND" H 5705 4127 50  0000 C CNN
 F 2 "" H 5700 4300 50  0001 C CNN
@@
 	6500 2400 6800 2400
 $Comp
-L Connector:Conn_01x03_Male J?
+L Connector:Conn_01x03_Male J1
 U 1 1 5DC9D3E0
 P 7000 2400
-F 0 "J?" H 6972 2332 50  0000 R CNN
+F 0 "J1" H 6972 2332 50  0000 R CNN
 F 1 "Conn_01x03_Male" H 6972 2423 50  0000 R CNN
-F 2 "" H 7000 2400 50  0001 C CNN
+F 2 "Connector_PinSocket_2.54mm:PinSocket_1x03_P2.54mm_Vertical" H 7000 2400 50  0001 C CNN
 F 3 "~" H 7000 2400 50  0001 C CNN
 	1    7000 2400
@@
 Connection ~ 5700 2800
 $Comp
-L power:GND #PWR?
+L power:GND #PWR0103
 U 1 1 5DC9E781
 P 6700 2600
-F 0 "#PWR?" H 6700 2350 50  0001 C CNN
+F 0 "#PWR0103" H 6700 2350 50  0001 C CNN
 F 1 "GND" H 6705 2427 50  0000 C CNN
 F 2 "" H 6700 2600 50  0001 C CNN
@@
 $EndComp
 $Comp
-L Device:R_Small R?
+L Device:R_Small R1
 U 1 1 5DC9ECDF
 P 7700 3100
-F 0 "R?" V 7504 3100 50  0000 C CNN
+F 0 "R1" V 7504 3100 50  0000 C CNN
 F 1 "100" V 7595 3100 50  0000 C CNN
-F 2 "" H 7700 3100 50  0001 C CNN
+F 2 "Resistor_SMD:R_0805_2012Metric" H 7700 3100 50  0001 C CNN
 F 3 "~" H 7700 3100 50  0001 C CNN
 	1    7700 3100
@@
 $EndComp
 $Comp
-L Device:R_Small R?
+L Device:R_Small R2
 U 1 1 5DC9F284
 P 7700 3500
-F 0 "R?" V 7504 3500 50  0000 C CNN
+F 0 "R2" V 7504 3500 50  0000 C CNN
 F 1 "100" V 7595 3500 50  0000 C CNN
-F 2 "" H 7700 3500 50  0001 C CNN
+F 2 "Resistor_SMD:R_0805_2012Metric" H 7700 3500 50  0001 C CNN
 F 3 "~" H 7700 3500 50  0001 C CNN
 	1    7700 3500
@@
 $EndComp
 $Comp
-L Device:R_Small R?
+L Device:R_Small R3
 U 1 1 5DC9F4CB
 P 7700 3900
-F 0 "R?" V 7504 3900 50  0000 C CNN
+F 0 "R3" V 7504 3900 50  0000 C CNN
 F 1 "100" V 7595 3900 50  0000 C CNN
-F 2 "" H 7700 3900 50  0001 C CNN
+F 2 "Resistor_SMD:R_0805_2012Metric" H 7700 3900 50  0001 C CNN
 F 3 "~" H 7700 3900 50  0001 C CNN
 	1    7700 3900
@@
 $EndComp
 $Comp
-L Device:LED_Small D?
+L Device:LED_Small D1
 U 1 1 5DC9FCAF
 P 8200 3300
-F 0 "D?" V 8246 3232 50  0000 R CNN
+F 0 "D1" V 8246 3232 50  0000 R CNN
 F 1 "LED" V 8155 3232 50  0000 R CNN
-F 2 "" V 8200 3300 50  0001 C CNN
+F 2 "janis:LED_2214A" V 8200 3300 50  0001 C CNN
 F 3 "~" V 8200 3300 50  0001 C CNN
 	1    8200 3300
@@
 $EndComp
 $Comp
-L Device:LED_Small D?
+L Device:LED_Small D2
 U 1 1 5DCA0D9E
 P 8200 3700
-F 0 "D?" V 8246 3632 50  0000 R CNN
+F 0 "D2" V 8246 3632 50  0000 R CNN
 F 1 "LED" V 8155 3632 50  0000 R CNN
-F 2 "" V 8200 3700 50  0001 C CNN
+F 2 "janis:LED_2214A" V 8200 3700 50  0001 C CNN
 F 3 "~" V 8200 3700 50  0001 C CNN
 	1    8200 3700
@@
 	8200 3100 8200 3200
 $Comp
-L Device:LED_Small D?
+L Device:LED_Small D3
 U 1 1 5DCA22F8
 P 8500 3300
-F 0 "D?" V 8454 3398 50  0000 L CNN
+F 0 "D3" V 8454 3398 50  0000 L CNN
 F 1 "LED" V 8545 3398 50  0000 L CNN
-F 2 "" V 8500 3300 50  0001 C CNN
+F 2 "janis:LED_2214A" V 8500 3300 50  0001 C CNN
 F 3 "~" V 8500 3300 50  0001 C CNN
 	1    8500 3300
@@
 $EndComp
 $Comp
-L Device:LED_Small D?
+L Device:LED_Small D4
 U 1 1 5DCA2835
 P 8500 3700
-F 0 "D?" V 8454 3798 50  0000 L CNN
+F 0 "D4" V 8454 3798 50  0000 L CNN
 F 1 "LED" V 8545 3798 50  0000 L CNN
-F 2 "" V 8500 3700 50  0001 C CNN
+F 2 "janis:LED_2214A" V 8500 3700 50  0001 C CNN
 F 3 "~" V 8500 3700 50  0001 C CNN
 	1    8500 3700
@@
 Connection ~ 8200 3900
 $Comp
-L Device:LED_Small D?
+L Device:LED_Small D5
 U 1 1 5DCA3D76
 P 8800 3500
-F 0 "D?" V 8754 3598 50  0000 L CNN
+F 0 "D5" V 8754 3598 50  0000 L CNN
 F 1 "LED" V 8845 3598 50  0000 L CNN
-F 2 "" V 8800 3500 50  0001 C CNN
+F 2 "janis:LED_2214A" V 8800 3500 50  0001 C CNN
 F 3 "~" V 8800 3500 50  0001 C CNN
 	1    8800 3500
@@
 $EndComp
 $Comp
-L Device:LED_Small D?
+L Device:LED_Small D6
 U 1 1 5DCA4204
 P 9100 3500
-F 0 "D?" V 9146 3432 50  0000 R CNN
+F 0 "D6" V 9146 3432 50  0000 R CNN
 F 1 "LED" V 9055 3432 50  0000 R CNN
-F 2 "" V 9100 3500 50  0001 C CNN
+F 2 "janis:LED_2214A" V 9100 3500 50  0001 C CNN
 F 3 "~" V 9100 3500 50  0001 C CNN
 	1    9100 3500

Commit message: Finished schematic and PCB
Parts:
- removed J1: Conn_01x03_Male, Connector_PinSocket_2.54mm:PinSocket_1x03_P2.54mm_Vertical, symbol Connector:Conn_01x03_Male
- added C2, C3: 10uF, Capacitor_SMD:C_0805_2012Metric, symbol Device:C_Small
- added CON1, CON2, CON3, CON4: 1PIN, Raksts_Test:TestPoint_2.00mm, symbol raksts:1PIN
- added SW1: SWT-2, Button_Switch_SMD:SW_SPST_EVQQ2, symbol electromechanics_ingus:SWT-2
- D1, D2, D3, D4, D5, D6: footprint janis:LED_2214A -> janis:LED_3528
Connections:
- net GND: now also C2.2, C3.2, CON3.1, SW1.2
- net at BT1.1 (+), C1.1, U1.1 (VCC): now also C2.1, C3.1, CON1.1
- net at U1.2 (PA6): now also SW1.1
- net at U1.3 (PA7): now also CON4.1
- net at U1.6 (~RESET~/PA0): now also CON2.1
Other:
- moved on the sheet: BT1
Changed lines of the file:
@@
 L Device:Battery_Cell BT1
 U 1 1 5DC992B0
-P 3800 3500
-F 0 "BT1" H 3918 3596 50  0000 L CNN
-F 1 "Battery_Cell" H 3918 3505 50  0000 L CNN
-F 2 "Battery:BatteryHolder_Keystone_3002_1x2032" V 3800 3560 50  0001 C CNN
-F 3 "~" V 3800 3560 50  0001 C CNN
-	1    3800 3500
+P 3500 3500
+F 0 "BT1" H 3618 3596 50  0000 L CNN
+F 1 "Battery_Cell" H 3618 3505 50  0000 L CNN
+F 2 "Battery:BatteryHolder_Keystone_3002_1x2032" V 3500 3560 50  0001 C CNN
+F 3 "~" V 3500 3560 50  0001 C CNN
+	1    3500 3500
 	1    0    0    -1
 $EndComp
@@
 	4500 2800 5700 2800
 Wire Wire Line
-	4500 2800 3800 2800
-Wire Wire Line
-	3800 2800 3800 3300
+	4500 2800 4100 2800
+Wire Wire Line
+	3500 2800 3500 3300
 Connection ~ 4500 2800
 Wire Wire Line
 	5700 4100 5700 4200
 Wire Wire Line
-	5700 4200 3800 4200
-Wire Wire Line
-	3800 4200 3800 3600
+	5700 4200 3500 4200
+Wire Wire Line
+	3500 4200 3500 3600
 Wire Wire Line
 	4500 3100 4500 3200
@@
 	6300 3200 6500 3200
 Wire Wire Line
-	6500 3200 6500 2400
-Wire Wire Line
-	6500 2400 6800 2400
-$Comp
-L Connector:Conn_01x03_Male J1
-U 1 1 5DC9D3E0
-P 7000 2400
-F 0 "J1" H 6972 2332 50  0000 R CNN
-F 1 "Conn_01x03_Male" H 6972 2423 50  0000 R CNN
-F 2 "Connector_PinSocket_2.54mm:PinSocket_1x03_P2.54mm_Vertical" H 7000 2400 50  0001 C CNN
-F 3 "~" H 7000 2400 50  0001 C CNN
-	1    7000 2400
-	-1   0    0    1
-$EndComp
+	6500 3200 6500 2300
+Wire Wire Line
+	6500 2300 6800 2300
 Wire Wire Line
 	6800 2500 6700 2500
@@
 	6700 2500 6700 2600
 Wire Wire Line
-	6800 2300 5700 2300
-Wire Wire Line
-	5700 2300 5700 2800
+	6800 2100 5700 2100
+Wire Wire Line
+	5700 2100 5700 2800
 Connection ~ 5700 2800
 $Comp
@@
 F 0 "D1" V 8246 3232 50  0000 R CNN
 F 1 "LED" V 8155 3232 50  0000 R CNN
-F 2 "janis:LED_2214A" V 8200 3300 50  0001 C CNN
+F 2 "janis:LED_3528" V 8200 3300 50  0001 C CNN
 F 3 "~" V 8200 3300 50  0001 C CNN
 	1    8200 3300
@@
 F 0 "D2" V 8246 3632 50  0000 R CNN
 F 1 "LED" V 8155 3632 50  0000 R CNN
-F 2 "janis:LED_2214A" V 8200 3700 50  0001 C CNN
+F 2 "janis:LED_3528" V 8200 3700 50  0001 C CNN
 F 3 "~" V 8200 3700 50  0001 C CNN
 	1    8200 3700
@@
 F 0 "D3" V 8454 3398 50  0000 L CNN
 F 1 "LED" V 8545 3398 50  0000 L CNN
-F 2 "janis:LED_2214A" V 8500 3300 50  0001 C CNN
+F 2 "janis:LED_3528" V 8500 3300 50  0001 C CNN
 F 3 "~" V 8500 3300 50  0001 C CNN
 	1    8500 3300
@@
 F 0 "D4" V 8454 3798 50  0000 L CNN
 F 1 "LED" V 8545 3798 50  0000 L CNN
-F 2 "janis:LED_2214A" V 8500 3700 50  0001 C CNN
+F 2 "janis:LED_3528" V 8500 3700 50  0001 C CNN
 F 3 "~" V 8500 3700 50  0001 C CNN
 	1    8500 3700
@@
 F 0 "D5" V 8754 3598 50  0000 L CNN
 F 1 "LED" V 8845 3598 50  0000 L CNN
-F 2 "janis:LED_2214A" V 8800 3500 50  0001 C CNN
+F 2 "janis:LED_3528" V 8800 3500 50  0001 C CNN
 F 3 "~" V 8800 3500 50  0001 C CNN
 	1    8800 3500
@@
 F 0 "D6" V 9146 3432 50  0000 R CNN
 F 1 "LED" V 9055 3432 50  0000 R CNN
-F 2 "janis:LED_2214A" V 9100 3500 50  0001 C CNN
+F 2 "janis:LED_3528" V 9100 3500 50  0001 C CNN
 F 3 "~" V 9100 3500 50  0001 C CNN
 	1    9100 3500
@@
 Wire Wire Line
 	7300 3900 7600 3900
+$Comp
+L raksts:1PIN CON1
+U 1 1 5DE8D4BC
+P 7000 2100
+F 0 "CON1" H 7128 2158 60  0000 L CNN
+F 1 "1PIN" H 7128 2052 60  0000 L CNN
+F 2 "Raksts_Test:TestPoint_2.00mm" H 7000 2100 60  0001 C CNN
+F 3 "" H 7000 2100 60  0000 C CNN
+	1    7000 2100
+	1    0    0    -1
+$EndComp
+$Comp
+L raksts:1PIN CON2
+U 1 1 5DE8DDE1
+P 7000 2300
+F 0 "CON2" H 7128 2358 60  0000 L CNN
+F 1 "1PIN" H 7128 2252 60  0000 L CNN
+F 2 "Raksts_Test:TestPoint_2.00mm" H 7000 2300 60  0001 C CNN
+F 3 "" H 7000 2300 60  0000 C CNN
+	1    7000 2300
+	1    0    0    -1
+$EndComp
+$Comp
+L raksts:1PIN CON3
+U 1 1 5DE8DF50
+P 7000 2500
+F 0 "CON3" H 7128 2558 60  0000 L CNN
+F 1 "1PIN" H 7128 2452 60  0000 L CNN
+F 2 "Raksts_Test:TestPoint_2.00mm" H 7000 2500 60  0001 C CNN
+F 3 "" H 7000 2500 60  0000 C CNN
+	1    7000 2500
+	1    0    0    -1
+$EndComp
+$Comp
+L power:GND #PWR0104
+U 1 1 5DE928DB
+P 7400 4500
+F 0 "#PWR0104" H 7400 4250 50  0001 C CNN
+F 1 "GND" H 7405 4327 50  0000 C CNN
+F 2 "" H 7400 4500 50  0001 C CNN
+F 3 "" H 7400 4500 50  0001 C CNN
+	1    7400 4500
+	1    0    0    -1
+$EndComp
+Wire Wire Line
+	6700 4300 6600 4300
+$Comp
+L raksts:1PIN CON4
+U 1 1 5DE96BE7
+P 6900 3700
+F 0 "CON4" H 7028 3758 60  0000 L CNN
+F 1 "1PIN" H 7028 3652 60  0000 L CNN
+F 2 "Raksts_Test:TestPoint_2.00mm" H 6900 3700 60  0001 C CNN
+F 3 "" H 6900 3700 60  0000 C CNN
+	1    6900 3700
+	1    0    0    -1
+$EndComp
+Wire Wire Line
+	6600 3600 6300 3600
+$Comp
+L electromechanics_ingus:SWT-2 SW1
+U 1 1 5DE99C0F
+P 6700 4300
+F 0 "SW1" H 6900 4481 60  0000 C CNN
+F 1 "SWT-2" H 6750 4175 60  0001 L BNN
+F 2 "Button_Switch_SMD:SW_SPST_EVQQ2" H 6900 4200 60  0001 C CNN
+F 3 "" H 6700 4300 60  0000 C CNN
+	1    6700 4300
+	1    0    0    -1
+$EndComp
+Wire Wire Line
+	7100 4300 7400 4300
+Wire Wire Line
+	7400 4300 7400 4500
+Wire Wire Line
+	6300 3700 6700 3700
+Wire Wire Line
+	6600 3600 6600 4300
+$Comp
+L Device:C_Small C3
+U 1 1 5DEAB656
+P 4100 3000
+F 0 "C3" H 4192 3046 50  0000 L CNN
+F 1 "10uF" H 4192 2955 50  0000 L CNN
+F 2 "Capacitor_SMD:C_0805_2012Metric" H 4100 3000 50  0001 C CNN
+F 3 "~" H 4100 3000 50  0001 C CNN
+	1    4100 3000
+	1    0    0    -1
+$EndComp
+$Comp
+L Device:C_Small C2
+U 1 1 5DEABBEE
+P 3800 3000
+F 0 "C2" H 3892 3046 50  0000 L CNN
+F 1 "10uF" H 3892 2955 50  0000 L CNN
+F 2 "Capacitor_SMD:C_0805_2012Metric" H 3800 3000 50  0001 C CNN
+F 3 "~" H 3800 3000 50  0001 C CNN
+	1    3800 3000
+	1    0    0    -1
+$EndComp
+Wire Wire Line
+	3800 2900 3800 2800
+Connection ~ 3800 2800
+Wire Wire Line
+	3800 2800 3500 2800
+Wire Wire Line
+	4100 2900 4100 2800
+Connection ~ 4100 2800
+Wire Wire Line
+	4100 2800 3800 2800
+Wire Wire Line
+	3800 3100 3800 3200
+Wire Wire Line
+	3800 3200 4100 3200
+Wire Wire Line
+	4100 3200 4100 3100
+Wire Wire Line
+	4100 3200 4100 3300
+Connection ~ 4100 3200
+$Comp
+L power:GND #PWR0105
+U 1 1 5DEB1A08
+P 4100 3300
+F 0 "#PWR0105" H 4100 3050 50  0001 C CNN
+F 1 "GND" H 4105 3127 50  0000 C CNN
+F 2 "" H 4100 3300 50  0001 C CNN
+F 3 "" H 4100 3300 50  0001 C CNN
+	1    4100 3300
+	1    0    0    -1
+$EndComp
 $EndSCHEMATC
